Commit message: R1_Lite: tune IK and mount trajectories so cross-body mounts succeed.
Key fixes:
- URDF: gripper finger2 mimics finger1, parse_mimic enabled in converter so
  PhysX applies PhysxMimicJointAPI; gripper actuator now drives joint1 only.
- Policies: auto-compute TCP_offset from finger-pair midpoint in link6 frame
  (replaces R1-tuned 0.0079/0.0908 hardcoded offsets that misaligned R1_Lite).
- Mount orientation fixed to [0.7071, 0, 0.7071, 0] (link6 +X -> world -Z) for
  R1_Lite; the R1 value [0, -1, 0, 0] aimed the gripper horizontally.
- DLS damping lambda_val raised 0.01 -> 0.10 so the IK doesn't snap when j4
  saturates on across-body reaches; eliminates the gear-throwing event.
- Mount swing uses smoothstep target interpolation (1.5 s, hold-at-end);
  descent ramps Z linearly over 1.5 s. Both prevent abrupt target steps.
- Initial arm pose pre-folds j3 to bias DLS toward the elbow-folded branch.

Test scaffolding:
- DEBUG_FIXED_OBJECT_XY in galaxea_lab_external_env replaces gear randomization
  with deterministic positions for repeatable IK debugging.
- Per-step IK diagnostic prints target/EE/gear/carrier/gripper for the active
  arm, throttled to 10 sim steps.
- Viewport camera and grasping height tuned for R1_Lite.

Co-Authored-By: Claude Opus 4.7 (1M context) <noreply@anthropic.com>

File: source/Galaxea_Lab_External/assets/Robots/R1_Lite/urdf/mmp_revB_invconfig_upright_a1x.urdf (robot description, URDF)
Before this commit: robot mmp_revB_invconfig_upright_a1x, 34 links, 33 joints
Joints:
- joint left_gripper_finger_joint2: mimic (none) -> joint=left_gripper_finger_joint1 multiplier=-1.0 offset=0.0
- joint right_gripper_finger_joint2: mimic (none) -> joint=right_gripper_finger_joint1 multiplier=-1.0 offset=0.0
