Commit message: Added automatic scripts for r1lite and r1pro datageneration. Also made modifications to model assets and scoring criteria.

File: source/Galaxea_Lab_External/assets/Robots/R1_Pro/urdf/r1pro_2026.urdf (robot description, URDF)
Before this commit: robot r1pro_urdf, 43 links, 42 joints
Links:
- removed link left_gmsl_link
- removed link right_gmsl_link
Joints:
- removed joint left_gmsl_joint
- removed joint right_gmsl_joint
